File: KiCAD/odb225ant.kicad_pcb (KiCad board)
At the start: 2 copper layers, 20 x 60 mm, 13 parts, among them J1 Conn_Coaxial, Q1 BF545A, Q2 BF245A

Commit message: Calcutated resistor values for power 5V and 3.3V
Parts:
- C5: value 10nF -> 100nF
- R1: value 100R -> 470R
- R2: value 1k -> 1k2
Connections:
- C4 pad 2: <NO NET> -> GND
Routing:
- net GND: vias 16 -> 17
