File: KiCAD/odb225ant.kicad_sch (KiCad schematic)
At the start: 13 parts, among them J1 Conn_Coaxial, Q1 BF545A, Q2 BF245A

Commit message: Calcutated resistor values for power 5V and 3.3V
Parts:
- C5: value 10nF -> 100nF
- R1: value 100R -> 470R
- R2: value 1k -> 1k2
Other:
- note added: "for power = 5V R1 = 560 or 620R R2 = 680R for power = 3.3V R1 = 1k2 R2 = 470R"
